Commit message: reduce camera weight to prevent the robot from wobbling; slow down epsilon decay

File: thesis_ws/src/turtlebot3/turtlebot3/turtlebot3_description/urdf/turtlebot3_burger.urdf.xacro (robot description, xacro)
@@ -193,5 +193,5 @@
     <inertial>
       <origin xyz="0 0 0" />
-      <mass value="0.095" />
+      <mass value="0.025" />
       <inertia ixx="0.0001" ixy="0.0" ixz="0.0"
                iyy="0.0001" iyz="0.0"
